Commit message: update

File: description/gps.xacro (robot description, xacro)
@@ -1,26 +1,23 @@
 <?xml version="1.0"?>
-<robot xmlns:xacro="http://www.ros.org/wiki/xacro" >
-    <joint name="gps_joint" type="fixed">
-        <parent link="chassis"/>
-        <child link="gps_link"/>
-        <origin xyz="0.1675 0.035 0.144" rpy="0 0 0"/>
-    </joint>
-    <link name="gps_link">
-        <visual>
-            <geometry>
-                <box size="0.03 0.03 0.01"/>
-            </geometry>
-            <material name="black"/>
-        </visual>
-    </link>
-    <gazebo reference="gps_link">
-      <selfCollide>false</selfCollide>
-    </gazebo>
-    <gazebo reference="gps_link">
-        <material>Gazebo/Red</material>
-        <sensor name="navsat_sensor" type="navsat">
-            <always_on>1</always_on>
-            <update_rate>30</update_rate>
-        </sensor>
-    </gazebo>
+<robot xmlns:xacro="http://www.ros.org/wiki/xacro">
+  <joint name="gps_joint" type="fixed">
+    <parent link="chassis"/>
+    <child link="gps_link"/>
+    <origin xyz="0.1675 0.035 0.144" rpy="0 0 0"/>
+  </joint>
+  <link name="gps_link">
+    <visual>
+      <geometry>
+        <box size="0.03 0.03 0.01"/>
+      </geometry>
+      <material name="black"/>
+    </visual>
+  </link>
+  <gazebo reference="gps_link">
+    <sensor name="navsat_sensor" type="navsat">
+      <always_on>true</always_on>
+      <update_rate>30</update_rate>
+      <topic>/gps</topic>
+    </sensor>
+  </gazebo>
 </robot>

File: description/magnetometer.xacro (robot description, xacro)
@@ -1,46 +1,24 @@
 <?xml version="1.0"?>
-<robot xmlns:xacro="http://www.ros.org/wiki/xacro" >
-    <joint name="magnetometer_joint" type="fixed">
-        <parent link="chassis"/>
-        <child link="magnetometer_link"/>
-        <origin xyz="0.1675 0 0.144" rpy="0 0 0"/>
-    </joint>
-    <link name="magnetometer_link">
-        <visual>
-            <geometry>
-                <box size="0.03 0.03 0.01"/>
-            </geometry>
-            <material name="black"/>
-        </visual>
-    </link>
-    <gazebo reference="magnetometer_link">
-      <selfCollide>false</selfCollide>
-    </gazebo>
-    <gazebo reference="magnetometer_link">
-        <material>Gazebo/Gray</material>
-        <sensor name="magnetometer" type="magnetometer">
-            <always_on>1</always_on>
-            <update_rate>50</update_rate>
-            <magnetometer>
-            <x>
-                <noise type="gaussian">
-                <mean>0.000000080</mean>
-                <bias_mean>0.000000400</bias_mean>
-                </noise>
-            </x>
-            <y>
-                <noise type="gaussian">
-                <mean>0.000000080</mean>
-                <bias_mean>0.000000400</bias_mean>
-                </noise>
-            </y>
-            <z>
-                <noise type="gaussian">
-                <mean>0.000000080</mean>
-                <bias_mean>0.000000400</bias_mean>
-                </noise>
-            </z>
-            </magnetometer>
-        </sensor>
-    </gazebo>
+<robot xmlns:xacro="http://www.ros.org/wiki/xacro">
+  <joint name="magnetometer_joint" type="fixed">
+    <parent link="chassis"/>
+    <child link="magnetometer_link"/>
+    <origin xyz="0.1675 0 0.144" rpy="0 0 0"/>
+  </joint>
+  <link name="magnetometer_link">
+    <visual>
+      <geometry>
+        <box size="0.03 0.03 0.01"/>
+      </geometry>
+      <material name="black"/>
+    </visual>
+  </link>
+  <!-- Gazebo moderno -->
+  <gazebo reference="magnetometer_link">
+    <sensor name="magnetometer" type="magnetometer">
+      <always_on>true</always_on>
+      <update_rate>50</update_rate>
+      <topic>/mag</topic>
+    </sensor>
+  </gazebo>
 </robot>

File: description/robot.urdf.xacro (robot description, xacro)
@@ -10,5 +10,5 @@
         <xacro:include filename="gazebo_control.xacro" />
     </xacro:unless>
-    <xacro:include filename="lidar.xacro" />
+    <!-- <xacro:include filename="lidar.xacro" /> -->
     <xacro:include filename="camera.xacro" />
     <!-- <xacro:include filename="depth_camera.xacro" /> -->
